File: roverwiring2022.kicad_sch (KiCad schematic)
At the start: 20 parts, among them J1 Conn_01x19, J10 Conn_01x05, J11 Conn_01x05, J12 Conn_01x05, J13 Conn_01x05, J2 Conn_01x19, J3 Conn_01x09, J4 Conn_01x04, J5 Conn_01x04, J6 Conn_01x04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

Commit message: resolved all outstanding drc conflicts and finished VCC and GND planes
Parts:
- BT1: value 24V -> 12V
Connections:
- net GND: now also J1.18 (Pin_18)
Changed lines of the file:
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@@
+    (effects (font (size 1.27 1.27)) (justify left bottom))
+  )
+  (label "GND" (at 214.63 71.12 0)
     (effects (font (size 1.27 1.27)) (justify left bottom))
   )
@@
       (effects (font (size 1.27 1.27)) (justify left))
     )
-    (property "Value" "24V" (id 1) (at 196.85 125.73 90)
+    (property "Value" "12V" (id 1) (at 196.85 125.73 90)
       (effects (font (size 1.27 1.27)) (justify left))
     )
@@
     )
     (path "/7be0d89d-6acb-4975-9cf3-573cdcfcf128"
-      (reference "BT1") (unit 1) (value "24V") (footprint "Connector_BarrelJack:BarrelJack_CLIFF_FC681465S_SMT_Horizontal")
+      (reference "BT1") (unit 1) (value "12V") (footprint "Connector_BarrelJack:BarrelJack_CLIFF_FC681465S_SMT_Horizontal")
     )
     (path "/fbcc7916-b404-4e1b-ae53-81b82c5cd4a3"
